File: Código Fuente/Teorema de Thevenin.brd (EAGLE design)
At the start: 56.8 x 53.3 mm, 13 parts, among them P1 12V, P2 2V, P3 5.06V

Commit message: Add files via upload
Parts:
- removed R8: 299‎Ω, AUTODESK_CIRCUITS_BREADBOARD:0207/10
- added Rpot1: 299‎Ω, AUTODESK_CIRCUITS_BREADBOARD:B25V
- moved P3 50.8 mm to (5.00, 175.2)
- moved R6 38.1 mm to (5.00, 124.4)
- moved Meter2 25.4 mm to (5.00, 149.8)
- moved R5 25.4 mm to (5.00, 111.7)
- moved Meter1 12.7 mm to (5.00, 162.5)
Connections:
- removed net N$7 (its old number): Meter1.+, R6.2, R8.2
- new net N$10: Rpot1.A
- new net N$11: Meter1.+, R6.2, Rpot1.S
- new net N$9: P3.2, Rpot1.E
- net N$1: no longer P3.2, R8.1
